Commit message: Add 1.2.2-dev release files.

File: denso_cobotta_descriptions/cobotta_description/cobotta.urdf.xacro (robot description, xacro)
@@ -3,7 +3,32 @@
 	<xacro:arg name="gripper_type" default="parallel"/>
 	<xacro:property name="gripper_type" value="$(arg gripper_type)" />
+	<xacro:property name="joint_damping" value="0.001" />
+	<xacro:property name="joint_friction" value="0.61" />
+	<!-- Mass of Links
+		NOTE: These are roughly estimated values.
+	-->
+	<xacro:property name="base_mass" value="1.4" />
+	<xacro:property name="J1_mass" value="1.29" />
+	<xacro:property name="J2_mass" value="0.39" />
+	<xacro:property name="J3_mass" value="0.35" />
+	<xacro:property name="J4_mass" value="0.35" />
+	<xacro:property name="J5_mass" value="0.19" />
+	<xacro:property name="J6_mass" value="0.03" />
+	<!-- Macro for calculating inertial matrix-->
+	<xacro:macro name="inertia_macro" params="radius height mass *origin">
+    	<inertial>
+    	  <mass value="${mass}" />
+		  <xacro:insert_block name="origin" />
+    	  <inertia ixx="${((1 / 4) * mass * radius * radius) + ((1 / 12) * mass * height * height)}" ixy="0.0" ixz="0.0"
+    	    iyy="${((1 / 4) * mass * radius * radius) + ((1 / 12) * mass * height * height)}" iyz="0.0"
+    	    izz="${(1 / 2) * mass * radius * radius}" />
+    	</inertial>
+  	</xacro:macro>
+	<!-- plugin for Gazebo -->
 	<gazebo>
 		<plugin name="gazebo_ros_control" filename="libgazebo_ros_control.so">
 			<robotNamespace>/cobotta</robotNamespace>
+      <robotSimType>gazebo_ros_control/DefaultRobotHWSim</robotSimType>
+      <legacyModeNS>true</legacyModeNS>
 		</plugin>
 	</gazebo>
@@ -26,9 +51,7 @@
 			</geometry>
 		</collision>
-		<inertial>
-			<mass value="1"/>
-			<origin rpy="0.000000 0.000000 0.000000" xyz="0.000000 0.000000 0.000000"/>
-			<inertia ixx="1" ixy="0" ixz="0" iyy="1" iyz="0" izz="1"/>
-		</inertial>
+		<xacro:inertia_macro radius="0.08" height="0.06" mass="${base_mass}">
+			<origin rpy="0.000000 0.000000 0.000000" xyz="-0.021310 0.000002 0.044011"/>
+		</xacro:inertia_macro>
 	</link>
 	<link name="J1">
@@ -45,25 +68,23 @@
 			</geometry>
 		</collision>
-		<inertial>
-			<mass value="1"/>
-			<origin rpy="0.000000 0.000000 0.000000" xyz="0.000000 0.000000 0.000000"/>
-			<inertia ixx="1" ixy="0" ixz="0" iyy="1" iyz="0" izz="1"/>
-		</inertial>
+		<xacro:inertia_macro radius="0.06" height="0.1" mass="${J1_mass}">
+			<origin rpy="0.000000 0.000000 0.000000" xyz="0.000000 0.000000 0.15" />
+		</xacro:inertia_macro>
 	</link>
 	<joint name="joint_1" type="revolute">
 		<parent link="base_link"/>
-		<child link="J1"/>
-		<origin rpy="0.000000 0.000000 0.000000" xyz="0.000000 0.000000 0.000000"/>
-		<axis xyz="-0.000000 -0.000000 1.000000"/>
-		<limit effort="1" lower="-2.617994" upper="2.617994" velocity="0.32253"/>
-		<dynamics damping="0" friction="0"/>
+		<child link="J1" />
+		<origin rpy="0.000000 0.000000 0.000000" xyz="0.000000 0.000000 0.000000" />
+		<axis xyz="-0.000000 -0.000000 1.000000" />
+		<limit effort="1" lower="-2.617994" upper="2.617994" velocity="0.40317105721069" />
+		<dynamics damping="${joint_damping}" friction="${joint_friction}" />
 	</joint>
 	<transmission name="trans_1">
 		<type>transmission_interface/SimpleTransmission</type>
 		<joint name="joint_1">
-			<hardwareInterface>PositionJointInterface</hardwareInterface>
+			<hardwareInterface>hardware_interface/PositionJointInterface</hardwareInterface>
 		</joint>
 		<actuator name="motor_1">
-			<hardwareInterface>PositionJointInterface</hardwareInterface>
+			<hardwareInterface>hardware_interface/PositionJointInterface</hardwareInterface>
 			<mechanicalReduction>1</mechanicalReduction>
 		</actuator>
@@ -82,25 +103,23 @@
 			</geometry>
 		</collision>
-		<inertial>
-			<mass value="1"/>
-			<origin rpy="0.000000 0.000000 0.000000" xyz="0.000000 0.000000 0.000000"/>
-			<inertia ixx="1" ixy="0" ixz="0" iyy="1" iyz="0" izz="1"/>
-		</inertial>
+		<xacro:inertia_macro radius="0.03" height="0.12" mass="${J2_mass}">
+			<origin rpy="0.000000 0.000000 0.000000" xyz="-0.020000 0.100000 0.070000" />
+		</xacro:inertia_macro>
 	</link>
 	<joint name="joint_2" type="revolute">
 		<parent link="J1"/>
 		<child link="J2"/>
-		<origin rpy="0.000000 0.000000 0.000000" xyz="0.000000 0.000000 0.180000"/>
-		<axis xyz="-0.000000 1.000000 -0.000000"/>
-		<limit effort="1" lower="-1.047198" upper="1.745329" velocity="0.31374"/>
-		<dynamics damping="0" friction="0"/>
+		<origin rpy="0.000000 0.000000 0.000000" xyz="0.000000 0.000000 0.180000" />
+		<axis xyz="-0.000000 1.000000 -0.000000" />
+		<limit effort="1" lower="-1.047198" upper="1.745329" velocity="0.392175482923126" />
+		<dynamics damping="${joint_damping}" friction="${joint_friction}"/>
 	</joint>
 	<transmission name="trans_2">
 		<type>transmission_interface/SimpleTransmission</type>
 		<joint name="joint_2">
-			<hardwareInterface>PositionJointInterface</hardwareInterface>
+			<hardwareInterface>hardware_interface/PositionJointInterface</hardwareInterface>
 		</joint>
 		<actuator name="motor_2">
-			<hardwareInterface>PositionJointInterface</hardwareInterface>
+			<hardwareInterface>hardware_interface/PositionJointInterface</hardwareInterface>
 			<mechanicalReduction>1</mechanicalReduction>
 		</actuator>
@@ -119,25 +138,23 @@
 			</geometry>
 		</collision>
-		<inertial>
-			<mass value="1"/>
-			<origin rpy="0.000000 0.000000 0.000000" xyz="0.000000 0.000000 0.000000"/>
-			<inertia ixx="1" ixy="0" ixz="0" iyy="1" iyz="0" izz="1"/>
-		</inertial>
+		<xacro:inertia_macro radius="0.03" height="0.11" mass="${J3_mass}">
+			<origin rpy="0.000000 0.000000 0.000000" xyz="-0.01000 0.020000 0.030000" />
+		</xacro:inertia_macro>
 	</link>
 	<joint name="joint_3" type="revolute">
 		<parent link="J2"/>
 		<child link="J3"/>
-		<origin rpy="0.000000 0.000000 0.000000" xyz="0.000000 0.000000 0.165000"/>
-		<axis xyz="-0.000000 1.000000 -0.000000"/>
-		<limit effort="1" lower="0.3141593" upper="2.443461" velocity="0.58056"/>
-		<dynamics damping="0" friction="0"/>
+		<origin rpy="0.000000 0.000000 0.000000" xyz="0.000000 0.000000 0.165000" />
+		<axis xyz="-0.000000 1.000000 -0.000000" />
+		<limit effort="1" lower="0.3141593" upper="2.443461" velocity="0.725707902979242" />
+		<dynamics damping="${joint_damping}" friction="${joint_friction}"/>
 	</joint>
 	<transmission name="trans_3">
 		<type>transmission_interface/SimpleTransmission</type>
 		<joint name="joint_3">
-			<hardwareInterface>PositionJointInterface</hardwareInterface>
+			<hardwareInterface>hardware_interface/PositionJointInterface</hardwareInterface>
 		</joint>
 		<actuator name="motor_3">
-			<hardwareInterface>PositionJointInterface</hardwareInterface>
+			<hardwareInterface>hardware_interface/PositionJointInterface</hardwareInterface>
 			<mechanicalReduction>1</mechanicalReduction>
 		</actuator>
@@ -145,5 +162,5 @@
 	<link name="J4">
 		<visual>
-			<origin rpy="0 0 0" xyz="0 0 -0.522500"/>
+			<origin rpy="0 0 0" xyz="0 0 0"/>
 			<geometry>
 				<mesh filename="package://denso_cobotta_descriptions/cobotta_description/J4.dae" scale="1 1 1"/>
@@ -156,25 +173,23 @@
 			</geometry>
 		</collision>
-		<inertial>
-			<mass value="1"/>
-			<origin rpy="0.000000 0.000000 0.000000" xyz="0.000000 0.000000 0.000000"/>
-			<inertia ixx="1" ixy="0" ixz="0" iyy="1" iyz="0" izz="1"/>
-		</inertial>
+		<xacro:inertia_macro radius="0.03" height="0.11" mass="${J4_mass}">
+			<origin rpy="0.000000 0.000000 0.000000" xyz="0.0000 0.000000 0.055000"/>
+		</xacro:inertia_macro>
 	</link>
 	<joint name="joint_4" type="revolute">
 		<parent link="J3"/>
 		<child link="J4"/>
-		<origin rpy="0.000000 0.000000 0.000000" xyz="-0.012000 0.020000 0.1775"/>
-		<axis xyz="-0.000000 -0.000000 1.000000"/>
-		<limit effort="1" lower="-2.96706" upper="2.96706" velocity="0.59131"/>
-		<dynamics damping="0" friction="0"/>
+		<origin rpy="0.000000 0.000000 0.000000" xyz="-0.012000 0.020000 0.088000" />
+		<axis xyz="-0.000000 -0.000000 1.000000" />
+		<limit effort="1" lower="-2.96706" upper="2.96706" velocity="0.739146938219599" />
+		<dynamics damping="${joint_damping}" friction="${joint_friction}"/>
 	</joint>
 	<transmission name="trans_4">
 		<type>transmission_interface/SimpleTransmission</type>
 		<joint name="joint_4">
-			<hardwareInterface>PositionJointInterface</hardwareInterface>
+			<hardwareInterface>hardware_interface/PositionJointInterface</hardwareInterface>
 		</joint>
 		<actuator name="motor_4">
-			<hardwareInterface>PositionJointInterface</hardwareInterface>
+			<hardwareInterface>hardware_interface/PositionJointInterface</hardwareInterface>
 			<mechanicalReduction>1</mechanicalReduction>
 		</actuator>
@@ -193,25 +208,23 @@
 			</geometry>
 		</collision>
-		<inertial>
-			<mass value="1"/>
-			<origin rpy="0.000000 0.000000 0.000000" xyz="0.000000 0.000000 0.000000"/>
-			<inertia ixx="1" ixy="0" ixz="0" iyy="1" iyz="0" izz="1"/>
-		</inertial>
+		<xacro:inertia_macro radius="0.03" height="0.06" mass="${J5_mass}">
+			<origin rpy="0.000000 0.000000 0.000000" xyz="0.000000 -0.040000 0.015000"/>
+		</xacro:inertia_macro>
 	</link>
 	<joint name="joint_5" type="revolute">
 		<parent link="J4"/>
 		<child link="J5"/>
-		<origin rpy="0.000000 0.000000 0.000000" xyz="0.000000 -0.020000 0.000000"/>
-		<axis xyz="-0.000000 1.000000 -0.000000"/>
-		<limit effort="1" lower="-1.658063" upper="2.356194" velocity="0.59131"/>
-		<dynamics damping="0" friction="0"/>
+		<origin rpy="0.000000 0.000000 0.000000" xyz="0.000000 -0.020000 0.089500" />
+		<axis xyz="-0.000000 1.000000 -0.000000" />
+		<limit effort="1" lower="-1.658063" upper="2.356194" velocity="0.739146938219599" />
+		<dynamics damping="${joint_damping}" friction="${joint_friction}"/>
 	</joint>
 	<transmission name="trans_5">
 		<type>transmission_interface/SimpleTransmission</type>
 		<joint name="joint_5">
-			<hardwareInterface>PositionJointInterface</hardwareInterface>
+			<hardwareInterface>hardware_interface/PositionJointInterface</hardwareInterface>
 		</joint>
 		<actuator name="motor_5">
-			<hardwareInterface>PositionJointInterface</hardwareInterface>
+			<hardwareInterface>hardware_interface/PositionJointInterface</hardwareInterface>
 			<mechanicalReduction>1</mechanicalReduction>
 		</actuator>
@@ -230,25 +243,23 @@
 			</geometry>
 		</collision>
-		<inertial>
-			<mass value="1"/>
-			<origin rpy="0.000000 0.000000 0.000000" xyz="0.000000 0.000000 0.000000"/>
-			<inertia ixx="1" ixy="0" ixz="0" iyy="1" iyz="0" izz="1"/>
-		</inertial>
+		<xacro:inertia_macro radius="0.03" height="0.01" mass="${J6_mass}">
+			<origin rpy="0.000000 0.000000 0.000000" xyz="0.000000 0.000000 0.000000" />
+		</xacro:inertia_macro>
 	</link>
 	<joint name="joint_6" type="revolute">
 		<parent link="J5"/>
 		<child link="J6"/>
-		<origin rpy="0.000000 0.000000 0.000000" xyz="0.000000 -0.044500 0.042000"/>
-		<axis xyz="-0.000000 -0.000000 1.000000"/>
-		<limit effort="1" lower="-2.96706" upper="2.96706" velocity="0.88746"/>
-		<dynamics damping="0" friction="0"/>
+		<origin rpy="0.000000 0.000000 0.000000" xyz="0.000000 -0.044500 0.042000" />
+		<axis xyz="-0.000000 -0.000000 1.000000" />
+		<limit effort="1" lower="-2.96706" upper="2.96706" velocity="1.1093312725676" />
+		<dynamics damping="${joint_damping}" friction="${joint_friction}"/>
 	</joint>
 	<transmission name="trans_6">
 		<type>transmission_interface/SimpleTransmission</type>
 		<joint name="joint_6">
-			<hardwareInterface>PositionJointInterface</hardwareInterface>
+			<hardwareInterface>hardware_interface/PositionJointInterface</hardwareInterface>
 		</joint>
 		<actuator name="motor_6">
-			<hardwareInterface>PositionJointInterface</hardwareInterface>
+			<hardwareInterface>hardware_interface/PositionJointInterface</hardwareInterface>
 			<mechanicalReduction>1</mechanicalReduction>
 		</actuator>

File: denso_cobotta_descriptions/cobotta_description/parallel.urdf.xacro (robot description, xacro)
@@ -49,5 +49,5 @@
 		<origin rpy="0.000000 0.000000 0.000000" xyz="0.000000 0.000000 0.06000"/>
 		<axis xyz="-0.000000 1.000000 -0.000000"/>
-		<limit effort="1" lower="0.000000" upper="0.015000" velocity="0.040000"/>
+		<limit effort="20" lower="0.000000" upper="0.015000" velocity="0.040000"/>
 		<dynamics damping="0" friction="0"/>
 	</joint>
@@ -55,8 +55,8 @@
 		<type>transmission_interface/SimpleTransmission</type>
 		<joint name="joint_gripper">
-			<hardwareInterface>PositionJointInterface</hardwareInterface>
+			<hardwareInterface>hardware_interface/PositionJointInterface</hardwareInterface>
 		</joint>
 		<actuator name="motor_gripper">
-			<hardwareInterface>PositionJointInterface</hardwareInterface>
+			<hardwareInterface>hardware_interface/PositionJointInterface</hardwareInterface>
 			<mechanicalReduction>1</mechanicalReduction>
 		</actuator>
@@ -87,6 +87,14 @@
 		<origin rpy="0.000000 0.000000 0.000000" xyz="0.000000 0.000000 0.060000"/>
 		<axis xyz="-0.000000 1.000000 -0.000000"/>
-		<limit effort="1" lower="-0.015000" upper="0.000000" velocity="0.040000"/>
+		<limit effort="20" lower="-0.015000" upper="0.000000" velocity="0.040000"/>
 		<dynamics damping="0" friction="0"/>
 	</joint>
+    	<!-- For gazebo simulation -->
+    	<gazebo>
+      	<plugin name="gripper_mimic_joint" filename="libroboticsgroup_gazebo_mimic_joint_plugin.so">
+        	<joint>joint_gripper</joint>
+        	<mimicJoint>joint_gripper_mimic</mimicJoint>
+        	<multiplier>-1</multiplier>
+      	</plugin>
+    	</gazebo>
 </robot>

File: denso_cobotta_moveit_config/config/cobotta.srdf.xacro (robot description, xacro)
@@ -14,5 +14,5 @@
     <!--SUBGROUPS: Groups can also be formed by referencing to already defined group names-->
     <group name="arm">
-	<link name="world" />
+	      <link name="world" />
         <link name="base_link" />
         <link name="J1" />
