Commit message: support  robot_description and robot_name in cobotta.body.urdf.xacro

File: denso_cobotta_descriptions/cobotta_description/cobotta.body.urdf.xacro (robot description, xacro)
@@ -2,5 +2,5 @@
 <robot name="cobotta" xmlns:xacro="http://www.ros.org/wiki/xacro">
   <xacro:macro name="cobotta_robot"
-               params="namespace">
+               params="namespace robot_description robot_name">
 	<!-- Parameters for gazebo simulation.
 		NOTE: These are roughly estimated values.
@@ -28,5 +28,6 @@
 	<gazebo>
 		<plugin name="gazebo_ros_control" filename="libgazebo_ros_control.so">
-			<robotNamespace>${namespace}/cobotta</robotNamespace>
+			<robotNamespace>${namespace}${robot_name}</robotNamespace>
+			<robotParam>${robot_description}</robotParam>
       <robotSimType>gazebo_ros_control/DefaultRobotHWSim</robotSimType>
       <legacyModeNS>true</legacyModeNS>

File: denso_cobotta_descriptions/cobotta_description/cobotta.urdf.xacro (robot description, xacro)
@@ -3,8 +3,14 @@
   <xacro:arg name="namespace" default=""/>
   <xacro:property name="namespace" value="$(arg namespace)" />
+  <xacro:arg name="robot_name" default="/cobotta"/>
+  <xacro:property name="robot_name" value="$(arg robot_name)" />
+  <xacro:arg name="robot_description" default="robot_description"/>
+  <xacro:property name="robot_description" value="$(arg robot_description)" />
   <xacro:arg name="gripper_type" default="parallel"/>
   <xacro:property name="gripper_type" value="$(arg gripper_type)" />
   <xacro:include filename="cobotta.body.urdf.xacro" />
-  <xacro:cobotta_robot namespace="${namespace}" />
+  <xacro:cobotta_robot namespace="${namespace}"
+                       robot_description="${robot_description}"
+                       robot_name="${robot_name}" />
   <xacro:if value="${gripper_type != 'none'}">
     <xacro:include filename="${gripper_type}.body.urdf.xacro" />
